Commit message: idefix_bringup + idefix_description: fix TF tree conflicts, scan yaw
Two TF conflicts found and fixed while wiring up robot_state_publisher
alongside the hardware LiDAR launch for the first time (previously
never run together, so these were latent, not active, until now).

base_footprint / base_link: odom_tf_broadcaster.py published
odom -> base_link directly, but the URDF has base_footprint as
base_link parent via a fixed joint (REP-105 pattern), so both were
claiming to be base_link parent. Retargeted odom_tf_broadcaster.py to
publish odom -> base_footprint instead. x/y/yaw are unaffected since
they come straight from wheel-encoder odometry either way; only z
differs between the two frames, and encoder odom z is always 0.

base_link / laser: renamed lidar_link to laser everywhere it appeared
(URDF link and joint child, Gazebo sensor reference and gz_frame_id,
both nav2_params.yaml costmap sensor_frame entries) so the frame name
matches what the real driver and static transform actually use.
Doing this exposed a second conflict: the URDF own lidar_joint still
carried its old placeholder origin, which now collided with
rplidar_c1.launch.py static transform for the same base_link -> laser
edge. Considered removing the URDF laser link entirely, rejected
because it would also remove Gazebo LiDAR sensor attachment point and
break sim. Fixed by syncing the URDF joint origin to match the launch
file value exactly; the two are kept in sync by convention (commented
in both files), not a single source of truth.

Scan yaw: rplidar_c1.launch.py static transform had no rotation
argument at all before this (defaulted to identity). Added one, first
set to yaw=pi per an initial assumption that the LiDAR sits rotated
180 degrees on its mount. Motion-tested by teleop: forward-detected
objects appeared behind the robot in the live map, so that assumption
was wrong. Reverted to yaw=0 (no rotational offset needed) in both
rplidar_c1.launch.py and the URDF joint it is kept in sync with.
Rebuilt, relaunched; not yet re-confirmed by a fresh teleop+RViz check
after this specific revert.

File: ros2_ws/idefix_description/urdf/idefix.gazebo.xacro (robot description, xacro)
@@ -21,9 +21,9 @@
     <mu2>0.0</mu2>
   </gazebo>
-  <gazebo reference="lidar_link">
+  <gazebo reference="laser">
   <sensor name="rplidar_c1" type="gpu_lidar">
     <topic>scan</topic>
     <update_rate>${lidar_rate_hz}</update_rate>
-    <gz_frame_id>lidar_link</gz_frame_id>
+    <gz_frame_id>laser</gz_frame_id>
     <alwaysOn>true</alwaysOn>
     <visualize>true</visualize>

File: ros2_ws/idefix_description/urdf/idefix.urdf.xacro (robot description, xacro)
@@ -157,5 +157,5 @@
   </joint>
   <!-- ===== sensors (all referenced to base_link) ===== -->
-  <link name="lidar_link">
+  <link name="laser">
     <visual>
       <geometry><cylinder radius="0.035" length="0.04"/></geometry>
@@ -169,6 +169,10 @@
   <joint name="lidar_joint" type="fixed">
     <parent link="base_link"/>
-    <child link="lidar_link"/>
-    <origin xyz="0 0 ${2*floor_gap + 0.025}" rpy="0 0 0"/> <!-- scan origin -->
+    <child link="laser"/>
+    <!-- Matches idefix_bringup's rplidar_c1.launch.py static transform exactly:
+         93mm deck stack + 35mm measured to the scan-plane slit, +/- 10mm
+         uncertainty. yaw=0: motion-tested on hardware, no rotational offset
+         needed. Keep both in sync. -->
+    <origin xyz="0 0 0.125" rpy="0 0 0"/>
   </joint>
   <link name="camera_link">
