Commit message: idefix_bringup: hardware speed limits, SLAM on rotation, LiDAR yaw
- slam_nav: Nav2 limited to 0.07 m/s and 0.5-0.6 rad/s to match the
  0.24 duty clamp (~0.085 m/s top speed); shared nav2_params.yaml keeps
  the sim tuning. Progress checker radius 0.5 -> 0.25 m.
- slam_toolbox_mapping: check_min_dist_and_heading_precisely so in-place
  turns trigger scan matching; travel thresholds 0.5 -> 0.2 m / rad.
- base_link -> laser yaw -8.1 deg, measured by straight-drive ICP
  (launch static TF and URDF lidar_joint).
- URDF track_width 0.216 -> 0.225 m (measured).
- slam_mapping docstring: map_saver_cli lives in nav2_map_server.

File: ros2_ws/idefix_description/urdf/idefix.urdf.xacro (robot description, xacro)
@@ -4,5 +4,5 @@
   <xacro:property name="wheel_radius"  value="0.022"/>   <!-- 44 mm dia -->
   <xacro:property name="wheel_width"   value="0.017"/>
-  <xacro:property name="track_width"   value="0.216"/>   <!-- TODO measure contact-to-contact on assembly; = plugin wheel_separation -->
+  <xacro:property name="track_width"   value="0.225"/>   <!-- measured wheel centre to wheel centre on the assembly; = plugin wheel_separation. Firmware WHEEL_BASE_M uses the effective 0.230 (tire scrub) -->
   <!-- ===== CHASSIS (radius is corrected diameter/2; confirm after measuring motor length) ===== -->
   <xacro:property name="base_radius"    value="0.125"/>  <!-- ~250 mm plate -->
@@ -172,7 +172,7 @@
     <!-- Matches idefix_bringup's rplidar_c1.launch.py static transform exactly:
          93mm deck stack + 35mm measured to the scan-plane slit, +/- 10mm
-         uncertainty. yaw=0: motion-tested on hardware, no rotational offset
-         needed. Keep both in sync. -->
-    <origin xyz="0 0 0.125" rpy="0 0 0"/>
+         uncertainty. yaw=-8.1deg: measured by straight-drive scan matching,
+         see rplidar_c1.launch.py. Keep both in sync. -->
+    <origin xyz="0 0 0.125" rpy="0 0 -0.1414"/>
   </joint>
   <link name="camera_link">
